File: pcb/Ethernet_interface.kicad_sch (KiCad schematic)
At the start: 32 parts, among them J1 RJ45_Hanrun_HR911105A_Horizon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, U1 W5500, Y1 25MHz

Commit message: Added cad and fixed small pcb issues
Parts:
- C1: LCSC (none) -> C1705
- C10, C11, C12, C13, C14, C16, C9: LCSC (none) -> C1525
- C2, C7: LCSC (none) -> C15195
- C3, C4: LCSC (none) -> C2186903
- C5, C8: LCSC (none) -> C318580
- C6: LCSC (none) -> C337699
- J2: LCSC (none) -> -
- R1: LCSC (none) -> C138060
- R10: LCSC (none) -> C138066
- R11: LCSC (none) -> C2909306
- R12: LCSC (none) -> C114759
- R2: LCSC (none) -> C138033
- R4, R5: LCSC (none) -> C105875
- R6, R7, R8, R9: LCSC (none) -> C87044
